Commit message: Update myrobot.xacro

File: urdf/myrobot.xacro (robot description, xacro)
@@ -135,5 +135,5 @@
       <origin xyz="0 0 0" rpy="0 0 0"/>
       <geometry>
-        <mesh filename="file://$(find ros2-lidar-object-detector)/meshes/lidar.dae"/>
+        <mesh filename="file://$(find lidar-object-follower)/meshes/lidar.dae"/>
       </geometry>
     </visual>

Commit message: Update myrobot.xacro

File: urdf/myrobot.xacro (robot description, xacro)
@@ -135,5 +135,5 @@
       <origin xyz="0 0 0" rpy="0 0 0"/>
       <geometry>
-        <mesh filename="file://$(find lidar-object-follower)/meshes/lidar.dae"/>
+        <mesh filename="file://$(find lidar_object_follower)/meshes/lidar.dae"/>
       </geometry>
     </visual>
